File: MCU Datalogger.kicad_sch (KiCad schematic)
At the start: 25 parts, among them U1 24LC1025, U2 DS1337S_, U3 24LC1025, U4 ATMEGA328P-AU, Y1 32.768 KHz, Y2 16 MHz

Commit message: Improved routing. Arranged values and ref. texts
Connections:
- net VCC: now also BT1.1 (+), C5.1, D2.2 (A), U4.18 (AVCC), U4.4 (VCC)
Changed lines of the file:
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@@
 	(wire
 		(pts
-			(xy 245.11 39.37) (xy 254 39.37)
+			(xy 245.11 39.37) (xy 270.51 39.37)
 		)
 		(stroke
@@
 		(pts
 			(xy 87.63 58.42) (xy 82.55 58.42)
-		)
-		(stroke
-			(width 0)
-			(type default)
-		)
-	)
-	(wire
-		(pts
-			(xy 270.51 39.37) (xy 254 39.37)
 		)
 		(stroke
@@
 		)
 	)
+	(label "VCC"
+		(at 261.62 39.37 0)
+		(fields_autoplaced yes)
+		(effects
+			(font
+				(size 1.27 1.27)
+			)
+			(justify left bottom)
+		)
+		(property "Net Class" "Power"
+			(at 261.62 40.64 0)
+			(hide yes)
+			(show_name no)
+			(do_not_autoplace no)
+			(effects
+				(font
+					(size 1.27 1.27)
+					(italic yes)
+				)
+				(justify left)
+			)
+		)
+	)

Commit message: Fixed two defects in the schematic
Connections:
- net SCK: no longer R3.2, U1.6 (SCL), U2.6 (SCL), U3.6 (SCL), U4.28 (PC5)
- new net SCL: R3.2, U1.6 (SCL), U2.6 (SCL), U3.6 (SCL), U4.28 (PC5)
Other:
- sheet Connectors ports: added SCL; removed none
Changed lines of the file:
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@@
 	(wire
 		(pts
-			(xy 245.11 31.75) (xy 245.11 39.37)
-		)
-		(stroke
-			(width 0)
-			(type default)
-		)
-	)
-	(wire
-		(pts
 			(xy 173.99 59.69) (xy 173.99 63.5)
 		)
@@
 		)
 	)
-	(label "SCK"
+	(label "SCL"
 		(at 85.09 138.43 0)
 		(effects
@@
 		)
 	)
-	(label "SCK"
-		(at 97.79 148.59 180)
-		(effects
-			(font
-				(size 1.27 1.27)
-			)
-			(justify right bottom)
-		)
-	)
 	(label "TX"
 		(at 226.06 49.53 0)
@@
 		)
 	)
+	(label "SCL"
+		(at 50.8 138.43 0)
+		(effects
+			(font
+				(size 1.27 1.27)
+			)
+			(justify left bottom)
+		)
+	)
 	(label "D3"
 		(at 226.06 54.61 0)
@@
 		)
 	)
-	(label "SCK"
+	(label "SCL"
 		(at 195.58 82.55 180)
 		(effects
@@
 	)
 	(label "TX"
-		(at 165.1 135.89 180)
+		(at 165.1 134.62 180)
 		(effects
 			(font
@@
 		)
 	)
-	(label "SCK"
-		(at 46.99 55.88 180)
-		(effects
-			(font
-				(size 1.27 1.27)
-			)
-			(justify right bottom)
-		)
-	)
 	(label "RX"
 		(at 226.06 46.99 0)
@@
 		)
 	)
-	(label "SCK"
-		(at 50.8 138.43 0)
-		(effects
-			(font
-				(size 1.27 1.27)
-			)
-			(justify left bottom)
-		)
-	)
 	(label "VCC"
 		(at 104.14 121.92 0)
@@
 		)
 	)
-	(label "SCK"
+	(label "SCL"
 		(at 165.1 129.54 180)
 		(effects
@@
 	)
 	(label "RX"
-		(at 165.1 138.43 180)
+		(at 165.1 137.16 180)
 		(effects
 			(font
@@
 		)
 	)
+	(label "SCL"
+		(at 46.99 55.88 180)
+		(effects
+			(font
+				(size 1.27 1.27)
+			)
+			(justify right bottom)
+		)
+	)
 	(label "VCC"
 		(at 179.07 85.09 180)
@@
 		)
 	)
+	(label "SCK"
+		(at 165.1 142.24 180)
+		(effects
+			(font
+				(size 1.27 1.27)
+			)
+			(justify right bottom)
+		)
+	)
+	(label "SCL"
+		(at 97.79 148.59 180)
+		(effects
+			(font
+				(size 1.27 1.27)
+			)
+			(justify right bottom)
+		)
+	)
 	(label "D8"
 		(at 190.5 139.7 0)
@@
 	)
 	(symbol
-		(lib_id "power:PWR_FLAG")
-		(at 245.11 31.75 0)
-		(unit 1)
-		(body_style 1)
-		(exclude_from_sim no)
-		(in_bom yes)
-		(on_board yes)
-		(in_pos_files yes)
-		(dnp no)
-		(fields_autoplaced yes)
-		(property "Reference" "#FLG01"
-			(at 245.11 29.845 0)
-			(hide yes)
-			(show_name no)
-			(do_not_autoplace no)
-			(effects
-				(font
-					(size 1.27 1.27)
-				)
-			)
-		)
-		(property "Value" "PWR_FLAG"
-			(at 245.11 26.67 0)
-			(show_name no)
-			(do_not_autoplace no)
-			(effects
-				(font
-					(size 1.27 1.27)
-				)
-			)
-		)
-		(property "Footprint" ""
-			(at 245.11 31.75 0)
-			(hide yes)
-			(show_name no)
-			(do_not_autoplace no)
-			(effects
-				(font
-					(size 1.27 1.27)
-				)
-			)
-		)
-		(property "Datasheet" ""
-			(at 245.11 31.75 0)
-			(hide yes)
-			(show_name no)
-			(do_not_autoplace no)
-			(effects
-				(font
-					(size 1.27 1.27)
-				)
-			)
-		)
-		(property "Description" "Special symbol for telling ERC where power comes from"
-			(at 245.11 31.75 0)
-			(hide yes)
-			(show_name no)
-			(do_not_autoplace no)
-			(effects
-				(font
-					(size 1.27 1.27)
-				)
-			)
-		)
-		(pin "1"
-		)
-		(instances
-			(project "MCU Datalogger"
-				(path "/b6931e11-5ca4-40d2-8041-2a917f2b0362"
-					(reference "#FLG01")
-					(unit 1)
-				)
-			)
-		)
-	)
-	(symbol
 		(lib_id "power:GND")
 		(at 40.64 151.13 0)
@@
 		)
 		(pin "RX" input
-			(at 165.1 138.43 180)
-			(effects
-				(font
-					(size 1.27 1.27)
-				)
-				(justify left)
-			)
-		)
-		(pin "SCK" passive
-			(at 165.1 129.54 180)
+			(at 165.1 137.16 180)
 			(effects
 				(font
@@
 		)
 		(pin "TX" output
-			(at 165.1 135.89 180)
+			(at 165.1 134.62 180)
 			(effects
 				(font
@@
 			(effects
 				(font
+					(size 1.27 1.27)
+				)
+				(justify left)
+			)
+		)
+		(pin "SCK" passive
+			(at 165.1 142.24 180)
+			(effects
+				(font
+					(size 1.27 1.27)
+				)
+				(justify left)
+			)
+		)
+		(pin "SCL" passive
+			(at 165.1 129.54 180)
+			(effects
+				(font
