File: MCU Datalogger.kicad_sch (KiCad schematic)
At the start: 25 parts, among them U1 24LC1025, U2 DS1337S_, U3 24LC1025, U4 ATMEGA328P-AU, Y1 32.768 KHz, Y2 16 MHz

Commit message: Fixed net bugs in 4-layer version
Connections:
- net ABC123: no longer names the net of C4.2, U4.20 (AREF)
Changed lines of the file:
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@@
-		)
-	)
-	(label "ABC123"
-		(at 180.34 31.75 0)
-		(effects
-			(font
-				(size 1.27 1.27)
-			)
-			(justify left bottom)
 		)
 	)
