File: MCU Datalogger.kicad_pcb (KiCad board)
At the start: 2 copper layers, 52.8 x 34.3 mm, 30 parts, among them J1 Conn_01x04_Pin, J2 Conn_01x09_Pin, J3 Conn_01x04_Pin, J4 Conn_02x03_Odd_Even, U1 24LC1025, U2 DS1337S_, U3 24LC1025, U4 ATMEGA328P-AU, Y1 32.768 KHz, Y2 16 MHz

Commit message: Fixed 2-layer PCB
Parts:
- moved J1 0.36 mm to (79.7, 70.7)
Connections:
- J1 pad 4: /SCK -> /SCL
- R3 pad 2: /SCK -> /SCL
- U1 pad 6: /SCK -> /SCL
- U2 pad 6: /SCK -> /SCL
- U3 pad 6: /SCK -> /SCL
- U4 pad 28: /SCK -> /SCL
Routing:
- net /SCL: track 0.00 -> 66.5 mm, vias 0 -> 4
- net /SCK: track 86.2 -> 27.5 mm, vias 3 -> 1
- net /VCC: track 196.0 -> 194.7 mm
- net /RESET: track 25.5 -> 26.0 mm
